Commit message: 增加传感器数据关闭

File: src/unitree_guide/unitree_ros/robots/a1_description/xacro/gazebo.xacro (robot description, xacro)
@@ -55,73 +55,25 @@
         </sensor>
     </gazebo>
-    <!-- base_self position and orientation. -->
-    <gazebo>
-        <plugin name="p3d_base_trunk_pos_vel" filename="libgazebo_ros_p3d.so">
-            <alwaysOn>true</alwaysOn>
-            <update_rate>100</update_rate>
-            <bodyName>base</bodyName>
-            <topicName>ground_truth/base_trunk</topicName>
-            <frameName>trunk</frameName>
-            <xyzOffsets>0 0 0</xyzOffsets>
-            <rpyOffsets>0 0 0</rpyOffsets>
-        </plugin>
-    </gazebo>
-    <!-- base_w position and orientation. -->
-    <gazebo>
-        <plugin name="p3d_base_w_pos_vel" filename="libgazebo_ros_p3d.so">
-            <alwaysOn>true</alwaysOn>
-            <update_rate>100</update_rate>
-            <bodyName>base</bodyName>
-            <topicName>ground_truth/base_w</topicName>
-            <frameName>world</frameName>
-            <xyzOffsets>0 0 0</xyzOffsets>
-            <rpyOffsets>0 0 0</rpyOffsets>
-        </plugin>
-    </gazebo>
-    <!-- Foot position and vel. -->
-    <gazebo>
-        <plugin name="p3d_FL_foot_pos_vel" filename="libgazebo_ros_p3d.so">
-            <alwaysOn>true</alwaysOn>
-            <update_rate>100</update_rate>
-            <bodyName>FL_foot</bodyName>
-            <topicName>ground_truth/FL_foot</topicName>
-            <frameName>base</frameName>
-            <xyzOffsets>0 0 0</xyzOffsets>
-            <rpyOffsets>0 0 0</rpyOffsets>
-        </plugin>
-    </gazebo>
-    <gazebo>
-        <plugin name="p3d_FR_foot_pos_vel" filename="libgazebo_ros_p3d.so">
-            <alwaysOn>true</alwaysOn>
-            <update_rate>100</update_rate>
-            <bodyName>FR_foot</bodyName>
-            <topicName>ground_truth/FR_foot</topicName>
-            <frameName>base</frameName>
-            <xyzOffsets>0 0 0</xyzOffsets>
-            <rpyOffsets>0 0 0</rpyOffsets>
-        </plugin>
-    </gazebo>
-    <gazebo>
-        <plugin name="p3d_RL_foot_pos_vel" filename="libgazebo_ros_p3d.so">
-            <alwaysOn>true</alwaysOn>
-            <update_rate>100</update_rate>
-            <bodyName>RL_foot</bodyName>
-            <topicName>ground_truth/RL_foot</topicName>
-            <frameName>base</frameName>
-            <xyzOffsets>0 0 0</xyzOffsets>
-            <rpyOffsets>0 0 0</rpyOffsets>
-        </plugin>
-    </gazebo>
-    <gazebo>
-        <plugin name="p3d_RR_foot_pos_vel" filename="libgazebo_ros_p3d.so">
-            <alwaysOn>true</alwaysOn>
-            <update_rate>100</update_rate>
-            <bodyName>RR_foot</bodyName>
-            <topicName>ground_truth/RR_foot</topicName>
-            <frameName>base</frameName>
-            <xyzOffsets>0 0 0</xyzOffsets>
-            <rpyOffsets>0 0 0</rpyOffsets>
-        </plugin>
-    </gazebo>
+    <xacro:macro name="p3d_truth_plugin" params="plugin_name body_name topic_name frame_name">
+        <gazebo>
+            <plugin name="${plugin_name}" filename="libgazebo_ros_p3d.so">
+                <alwaysOn>true</alwaysOn>
+                <update_rate>100</update_rate>
+                <bodyName>${body_name}</bodyName>
+                <topicName>${topic_name}</topicName>
+                <frameName>${frame_name}</frameName>
+                <xyzOffsets>0 0 0</xyzOffsets>
+                <rpyOffsets>0 0 0</rpyOffsets>
+            </plugin>
+        </gazebo>
+    </xacro:macro>
+    <xacro:if value="$(arg ENABLE_GROUND_TRUTH)">
+        <xacro:p3d_truth_plugin plugin_name="p3d_base_trunk_pos_vel" body_name="base" topic_name="ground_truth/base_trunk" frame_name="trunk"/>
+        <xacro:p3d_truth_plugin plugin_name="p3d_base_w_pos_vel" body_name="base" topic_name="ground_truth/base_w" frame_name="world"/>
+        <xacro:p3d_truth_plugin plugin_name="p3d_FL_foot_pos_vel" body_name="FL_foot" topic_name="ground_truth/FL_foot" frame_name="base"/>
+        <xacro:p3d_truth_plugin plugin_name="p3d_FR_foot_pos_vel" body_name="FR_foot" topic_name="ground_truth/FR_foot" frame_name="base"/>
+        <xacro:p3d_truth_plugin plugin_name="p3d_RL_foot_pos_vel" body_name="RL_foot" topic_name="ground_truth/RL_foot" frame_name="base"/>
+        <xacro:p3d_truth_plugin plugin_name="p3d_RR_foot_pos_vel" body_name="RR_foot" topic_name="ground_truth/RR_foot" frame_name="base"/>
+    </xacro:if>
     <!-- Foot contacts. -->
     <gazebo reference="FR_calf">
@@ -318,39 +270,40 @@
         <kd  value="1.0"/>
     </gazebo>
-     <!-- gazebo livox mid360 plugins -->
-    <xacro:property name="M_PI" value="3.14159"/>
-    <gazebo reference="laser_livox">
-        <sensor type="ray" name="laser_livox">
-            <pose>0 0 0 0 0 0</pose>
-            <visualize>true</visualize>
-            <update_rate>10</update_rate>
-            <plugin name="gazebo_ros_laser_controller" filename="liblivox_laser_simulation.so">
-                            <ray>
-                            <scan>
-                                    <horizontal>
-                                    <samples>100</samples>
-                                    <resolution>1</resolution>
-                                    <min_angle>${0}</min_angle>
-                                    <max_angle>${2*M_PI}</max_angle>
-                                    </horizontal>
-                                    <vertical>
-                                    <samples>360</samples>
-                                    <resolution>1</resolution>
-                                    <min_angle>${-5.22/180*M_PI}</min_angle>
-                                    <max_angle>${57.22/180*M_PI}</max_angle>
-                                    </vertical>
-                            </scan>
-                            <range>
-                                    <min>0.1</min>
-                                    <max>40</max>
-                                    <resolution>0.01</resolution>
-                            </range>
-                            <noise>
-                                    <type>gaussian</type>
-                                    <mean>0.0</mean>
-                                    <stddev>0.005</stddev>
-                            </noise>
-                            </ray>
-            <visualize>true</visualize>
+    <xacro:if value="$(arg ENABLE_SENSOR_DATA)">
+        <!-- gazebo livox mid360 plugins -->
+        <xacro:property name="M_PI" value="3.14159"/>
+        <gazebo reference="laser_livox">
+            <sensor type="ray" name="laser_livox">
+                <pose>0 0 0 0 0 0</pose>
+                <visualize>true</visualize>
+                <update_rate>10</update_rate>
+                <plugin name="gazebo_ros_laser_controller" filename="liblivox_laser_simulation.so">
+                    <ray>
+                        <scan>
+                            <horizontal>
+                                <samples>100</samples>
+                                <resolution>1</resolution>
+                                <min_angle>${0}</min_angle>
+                                <max_angle>${2*M_PI}</max_angle>
+                            </horizontal>
+                            <vertical>
+                                <samples>360</samples>
+                                <resolution>1</resolution>
+                                <min_angle>${-5.22/180*M_PI}</min_angle>
+                                <max_angle>${57.22/180*M_PI}</max_angle>
+                            </vertical>
+                        </scan>
+                        <range>
+                            <min>0.1</min>
+                            <max>40</max>
+                            <resolution>0.01</resolution>
+                        </range>
+                        <noise>
+                            <type>gaussian</type>
+                            <mean>0.0</mean>
+                            <stddev>0.005</stddev>
+                        </noise>
+                    </ray>
+                    <visualize>true</visualize>
                     <samples>24000</samples>
                     <downsample>1</downsample>
@@ -358,69 +311,66 @@
                     <ros_topic>/scan</ros_topic>
                     <frameName>laser_livox</frameName>
-            </plugin>
-        </sensor>
-    </gazebo>
-    <!-- gazebo livox imu-link plugins -->
-    <gazebo reference="livox_imu_link">
-    <gravity>true</gravity>
-    <sensor name="imu_sensor" type="imu">
-        <always_on>true</always_on>
-        <update_rate>1000</update_rate>
-        <visualize>true</visualize>
-        <topic>__default_topic__</topic>
-        <plugin filename="libgazebo_ros_imu_sensor.so" name="imu_plugin">
-            <topicName>/livox/imu</topicName>
-            <bodyName>livox_imu_link</bodyName>
-            <updateRateHZ>1000.0</updateRateHZ>
-            <gaussianNoise>0.0</gaussianNoise>
-            <xyzOffset>0 0 0</xyzOffset>
-            <rpyOffset>0 0 0</rpyOffset>
-            <frameName>livox_imu_link</frameName>
-        </plugin>
-        <pose>0 0 0 0 0 0</pose>
-    </sensor>
-    </gazebo>
-    <!-- camera 单目相机插件 -->
-    <gazebo reference="front_camera">
-    <material>Gazebo/Grey</material>
-        <sensor type="camera" name="camera">
-        <update_rate>30.0</update_rate>
-        <camera name="head">
-            <horizontal_fov>1.3962634</horizontal_fov>
-            <image>
-            <width>800</width>
-            <height>800</height>
-            <format>R8G8B8</format>
-            </image>
-            <clip>
-            <near>0.02</near>
-            <far>300</far>
-            </clip>
-            <noise>
-            <type>gaussian</type>
-            <!-- Noise is sampled independently per pixel on each frame.
-                That pixel's noise value is added to each of its color
-                channels, which at that point lie in the range [0,1]. -->
-            <mean>0.0</mean>
-            <stddev>0.007</stddev>
-            </noise>
-        </camera>
-        <plugin name="camera_controller" filename="libgazebo_ros_camera.so">
-            <alwaysOn>true</alwaysOn>
-            <updateRate>0.0</updateRate>
-            <cameraName>camera</cameraName>
-            <imageTopicName>image_raw</imageTopicName>
-            <cameraInfoTopicName>camera_info</cameraInfoTopicName>
-            <frameName>front_camera</frameName>
-            <hackBaseline>0.07</hackBaseline>
-            <distortionK1>0.0</distortionK1>
-            <distortionK2>0.0</distortionK2>
-            <distortionK3>0.0</distortionK3>
-            <distortionT1>0.0</distortionT1>
-            <distortionT2>0.0</distortionT2>
-        </plugin>
-        </sensor>
+                </plugin>
+            </sensor>
         </gazebo>
-        <!-- real_sense  深度相机(kinect)插件 -->
+        <!-- gazebo livox imu-link plugins -->
+        <gazebo reference="livox_imu_link">
+            <gravity>true</gravity>
+            <sensor name="imu_sensor" type="imu">
+                <always_on>true</always_on>
+                <update_rate>1000</update_rate>
+                <visualize>true</visualize>
+                <topic>__default_topic__</topic>
+                <plugin filename="libgazebo_ros_imu_sensor.so" name="imu_plugin">
+                    <topicName>/livox/imu</topicName>
+                    <bodyName>livox_imu_link</bodyName>
+                    <updateRateHZ>1000.0</updateRateHZ>
+                    <gaussianNoise>0.0</gaussianNoise>
+                    <xyzOffset>0 0 0</xyzOffset>
+                    <rpyOffset>0 0 0</rpyOffset>
+                    <frameName>livox_imu_link</frameName>
+                </plugin>
+                <pose>0 0 0 0 0 0</pose>
+            </sensor>
+        </gazebo>
+        <!-- camera 单目相机插件 -->
+        <gazebo reference="front_camera">
+            <material>Gazebo/Grey</material>
+            <sensor type="camera" name="camera">
+                <update_rate>30.0</update_rate>
+                <camera name="head">
+                    <horizontal_fov>1.3962634</horizontal_fov>
+                    <image>
+                        <width>800</width>
+                        <height>800</height>
+                        <format>R8G8B8</format>
+                    </image>
+                    <clip>
+                        <near>0.02</near>
+                        <far>300</far>
+                    </clip>
+                    <noise>
+                        <type>gaussian</type>
+                        <mean>0.0</mean>
+                        <stddev>0.007</stddev>
+                    </noise>
+                </camera>
+                <plugin name="camera_controller" filename="libgazebo_ros_camera.so">
+                    <alwaysOn>true</alwaysOn>
+                    <updateRate>0.0</updateRate>
+                    <cameraName>camera</cameraName>
+                    <imageTopicName>image_raw</imageTopicName>
+                    <cameraInfoTopicName>camera_info</cameraInfoTopicName>
+                    <frameName>front_camera</frameName>
+                    <hackBaseline>0.07</hackBaseline>
+                    <distortionK1>0.0</distortionK1>
+                    <distortionK2>0.0</distortionK2>
+                    <distortionK3>0.0</distortionK3>
+                    <distortionT1>0.0</distortionT1>
+                    <distortionT2>0.0</distortionT2>
+                </plugin>
+            </sensor>
+        </gazebo>
+        <!-- real_sense 深度相机(kinect)插件 -->
         <gazebo reference="real_sense">
             <sensor type="depth" name="real_sense">
@@ -459,3 +409,4 @@
             </sensor>
         </gazebo>
+    </xacro:if>
 </robot>

File: src/unitree_guide/unitree_ros/robots/a1_description/xacro/robot.xacro (robot description, xacro)
@@ -2,4 +2,6 @@
 <robot name="a1" xmlns:xacro="http://www.ros.org/wiki/xacro">
     <xacro:arg name="DEBUG" default="false"/>
+    <xacro:arg name="ENABLE_SENSOR_DATA" default="true"/>
+    <xacro:arg name="ENABLE_GROUND_TRUTH" default="true"/>
     <xacro:include filename="$(find a1_description)/xacro/const.xacro"/>
     <xacro:include filename="$(find a1_description)/xacro/materials.xacro"/>
@@ -111,106 +113,82 @@
     </link>
     <!-- livox mid360 -->
-    <!-- 对于本体 -->
     <link name="laser_livox">
             <collision>
-            <origin xyz="0 0 0" rpy="0 0 0"/>
-            <geometry>
+                <origin xyz="0 0 0" rpy="0 0 0"/>
+                <geometry>
                     <mesh filename="package://a1_description/meshes/livox_mid360.dae"/>
-            </geometry>
-            </collision>
-            <visual>
-            <origin xyz="0.0 0 0" rpy="0 0 0"/>
-            <geometry>
+                </geometry>
+            </collision>
+            <visual>
+                <origin xyz="0.0 0 0" rpy="0 0 0"/>
+                <geometry>
                     <mesh filename="package://a1_description/meshes/livox_mid360.dae"/>
-            </geometry>
-            </visual>
-    </link>
-    <!-- 对于连接 -->
-    <joint name="laser_livox_joint" type="fixed" >
-        <origin xyz="0.2 0 0.08" rpy="0 0.785 0" />
-        <parent link="base" />
-        <child link="laser_livox"/>
+                </geometry>
+            </visual>
+    </link>
+    <joint name="laser_livox_joint" type="fixed">
+            <origin xyz="0.2 0 0.08" rpy="0 0.785 0"/>
+            <parent link="base"/>
+            <child link="laser_livox"/>
     </joint>
     <!-- livox mid360-imu -->
-    <!-- 对于本体 -->
     <link name="livox_imu_link">
-        <inertial>
-            <mass value="0.001"/>
-            <origin rpy="0 0 0" xyz="0 0 0"/>
-            <inertia ixx="0.0001" ixy="0" ixz="0" iyy="0.0001" iyz="0" izz="0.0001"/>
-        </inertial>
-        <visual>
-            <origin rpy="0 0 0" xyz="0 0 0"/>
-            <geometry>
-                <box size="0.001 0.001 0.001"/>
-            </geometry>
-            <!-- <material name="red"/> -->
-        </visual>
-        <collision>
-            <origin rpy="0 0 0" xyz="0 0 0"/>
-            <geometry>
-                <box size=".001 .001 .001"/>
-            </geometry>
-        </collision>
-    </link>
-     <!-- 对于连接 -->
-     <joint name="livox_imu_joint" type="fixed">
-        <parent link="laser_livox"/>
-        <child link="livox_imu_link"/>
-        <origin rpy="0 0 0" xyz="-0.011 -0.02329 0.04412"/>
-    </joint>
-    <!--深度相机-->
-    <link
-        name="real_sense">
-        <inertial>
-        <origin
-            xyz="-0.00975078931607951 0.00306064913353049 -7.04374991291334E-05"
-            rpy="0 0 0" />
-        <mass
-            value="0.103311749598955" />
-        <inertia
-            ixx="7.35323632954531E-05"
-            ixy="3.0437488683846E-06"
-            ixz="2.08538534427428E-08"
-            iyy="7.40427481540393E-06"
-            iyz="-1.93018760531168E-08"
-            izz="7.2832884533889E-05" />
-        </inertial>
-        <visual>
-        <origin
-            xyz="0 0 0"
-            rpy="0 0 1.5708" />
-        <geometry>
-            <mesh
-            filename="package://a1_description/meshes/d415.stl" />
-        </geometry>
-        <material
-            name="">
-            <color
-            rgba="0.666666666666667 0.698039215686274 0.768627450980392 1" />
-        </material>
-        </visual>
-        <collision>
-        <origin
-            xyz="0 0 0"
-            rpy="0 0 0" />
-        <geometry>
-            <mesh
-            filename="package://a1_description/meshes/d415.stl" />
-        </geometry>
-        </collision>
-    </link>
-    <joint
-        name="real_sense_joint"
-        type="fixed">
-        <origin
-        xyz="0.28 0 0.043"
-        rpy="0 0 0" />
-        <parent
-        link="base" />
-        <child
-        link="real_sense" />
-        <axis
-        xyz="0 0 1" />
+            <inertial>
+                <mass value="0.001"/>
+                <origin rpy="0 0 0" xyz="0 0 0"/>
+                <inertia ixx="0.0001" ixy="0" ixz="0" iyy="0.0001" iyz="0" izz="0.0001"/>
+            </inertial>
+            <visual>
+                <origin rpy="0 0 0" xyz="0 0 0"/>
+                <geometry>
+                    <box size="0.001 0.001 0.001"/>
+                </geometry>
+            </visual>
+            <collision>
+                <origin rpy="0 0 0" xyz="0 0 0"/>
+                <geometry>
+                    <box size=".001 .001 .001"/>
+                </geometry>
+            </collision>
+    </link>
+    <joint name="livox_imu_joint" type="fixed">
+            <parent link="laser_livox"/>
+            <child link="livox_imu_link"/>
+            <origin rpy="0 0 0" xyz="-0.011 -0.02329 0.04412"/>
+    </joint>
+    <!-- depth camera -->
+    <link name="real_sense">
+            <inertial>
+                <origin xyz="-0.00975078931607951 0.00306064913353049 -7.04374991291334E-05" rpy="0 0 0"/>
+                <mass value="0.103311749598955"/>
+                <inertia
+                    ixx="7.35323632954531E-05"
+                    ixy="3.0437488683846E-06"
+                    ixz="2.08538534427428E-08"
+                    iyy="7.40427481540393E-06"
+                    iyz="-1.93018760531168E-08"
+                    izz="7.2832884533889E-05"/>
+            </inertial>
+            <visual>
+                <origin xyz="0 0 0" rpy="0 0 1.5708"/>
+                <geometry>
+                    <mesh filename="package://a1_description/meshes/d415.stl"/>
+                </geometry>
+                <material name="">
+                    <color rgba="0.666666666666667 0.698039215686274 0.768627450980392 1"/>
+                </material>
+            </visual>
+            <collision>
+                <origin xyz="0 0 0" rpy="0 0 0"/>
+                <geometry>
+                    <mesh filename="package://a1_description/meshes/d415.stl"/>
+                </geometry>
+            </collision>
+    </link>
+    <joint name="real_sense_joint" type="fixed">
+            <origin xyz="0.28 0 0.043" rpy="0 0 0"/>
+            <parent link="base"/>
+            <child link="real_sense"/>
+            <axis xyz="0 0 1"/>
     </joint>
     <xacro:leg name="FR" mirror="-1" mirror_dae="False" front_hind="1" front_hind_dae="True">
