Commit message: 时间片优化

File: src/unitree_guide/unitree_ros/robots/a1_description/xacro/gazebo.xacro (robot description, xacro)
@@ -113,33 +113,35 @@
         </sensor>
     </gazebo>
-    <!-- Visualization of Foot contacts. -->
-    <gazebo reference="FR_foot">
-        <visual>
-            <plugin name="drawForcePlugin" filename="libunitreeDrawForcePlugin.so">
-                <topicName>FR_foot_contact</topicName>
-            </plugin>
-        </visual>
-    </gazebo>
-    <gazebo reference="FL_foot">
-        <visual>
-            <plugin name="drawForcePlugin" filename="libunitreeDrawForcePlugin.so">
-                <topicName>FL_foot_contact</topicName>
-            </plugin>
-        </visual>
-    </gazebo>
-    <gazebo reference="RR_foot">
-        <visual>
-            <plugin name="drawForcePlugin" filename="libunitreeDrawForcePlugin.so">
-                <topicName>RR_foot_contact</topicName>
-            </plugin>
-        </visual>
-    </gazebo>
-    <gazebo reference="RL_foot">
-        <visual>
-            <plugin name="drawForcePlugin" filename="libunitreeDrawForcePlugin.so">
-                <topicName>RL_foot_contact</topicName>
-            </plugin>
-        </visual>
-    </gazebo>
+    <xacro:if value="$(arg ENABLE_FOOT_FORCE_VISUAL)">
+        <!-- Visualization of foot contacts. Disabled by default for competition scenes. -->
+        <gazebo reference="FR_foot">
+            <visual>
+                <plugin name="drawForcePlugin" filename="libunitreeDrawForcePlugin.so">
+                    <topicName>FR_foot_contact</topicName>
+                </plugin>
+            </visual>
+        </gazebo>
+        <gazebo reference="FL_foot">
+            <visual>
+                <plugin name="drawForcePlugin" filename="libunitreeDrawForcePlugin.so">
+                    <topicName>FL_foot_contact</topicName>
+                </plugin>
+            </visual>
+        </gazebo>
+        <gazebo reference="RR_foot">
+            <visual>
+                <plugin name="drawForcePlugin" filename="libunitreeDrawForcePlugin.so">
+                    <topicName>RR_foot_contact</topicName>
+                </plugin>
+            </visual>
+        </gazebo>
+        <gazebo reference="RL_foot">
+            <visual>
+                <plugin name="drawForcePlugin" filename="libunitreeDrawForcePlugin.so">
+                    <topicName>RL_foot_contact</topicName>
+                </plugin>
+            </visual>
+        </gazebo>
+    </xacro:if>
     <gazebo reference="base">
         <material>Gazebo/Green</material>

File: src/unitree_guide/unitree_ros/robots/a1_description/xacro/robot.xacro (robot description, xacro)
@@ -4,4 +4,5 @@
     <xacro:arg name="ENABLE_SENSOR_DATA" default="true"/>
     <xacro:arg name="ENABLE_GROUND_TRUTH" default="true"/>
+    <xacro:arg name="ENABLE_FOOT_FORCE_VISUAL" default="false"/>
     <xacro:include filename="$(find a1_description)/xacro/const.xacro"/>
     <xacro:include filename="$(find a1_description)/xacro/materials.xacro"/>
