Commit message: 电梯上下层BUG修复

File: src/unitree_guide/unitree_ros/robots/a1_description/xacro/gazebo.xacro (robot description, xacro)
@@ -68,5 +68,5 @@
         </gazebo>
     </xacro:macro>
-    <xacro:if value="$(arg ENABLE_GROUND_TRUTH)">
+    <xacro:if value="${'$(arg ENABLE_GROUND_TRUTH)' == 'true'}">
         <xacro:p3d_truth_plugin plugin_name="p3d_base_trunk_pos_vel" body_name="base" topic_name="ground_truth/base_trunk" frame_name="trunk"/>
         <xacro:p3d_truth_plugin plugin_name="p3d_base_w_pos_vel" body_name="base" topic_name="ground_truth/base_w" frame_name="world"/>
@@ -113,5 +113,5 @@
         </sensor>
     </gazebo>
-    <xacro:if value="$(arg ENABLE_FOOT_FORCE_VISUAL)">
+    <xacro:if value="${'$(arg ENABLE_FOOT_FORCE_VISUAL)' == 'true'}">
         <!-- Visualization of foot contacts. Disabled by default for competition scenes. -->
         <gazebo reference="FR_foot">
@@ -272,12 +272,39 @@
         <kd  value="1.0"/>
     </gazebo>
-    <xacro:if value="$(arg ENABLE_SENSOR_DATA)">
+    <xacro:if value="${'$(arg ENABLE_SENSOR_DATA)' == 'true'}">
         <!-- gazebo livox mid360 plugins -->
         <xacro:property name="M_PI" value="3.14159"/>
         <gazebo reference="laser_livox">
             <sensor type="ray" name="laser_livox">
+                <always_on>true</always_on>
                 <pose>0 0 0 0 0 0</pose>
                 <visualize>true</visualize>
                 <update_rate>10</update_rate>
+                <ray>
+                    <scan>
+                        <horizontal>
+                            <samples>100</samples>
+                            <resolution>1</resolution>
+                            <min_angle>${0}</min_angle>
+                            <max_angle>${2*M_PI}</max_angle>
+                        </horizontal>
+                        <vertical>
+                            <samples>360</samples>
+                            <resolution>1</resolution>
+                            <min_angle>${-5.22/180*M_PI}</min_angle>
+                            <max_angle>${57.22/180*M_PI}</max_angle>
+                        </vertical>
+                    </scan>
+                    <range>
+                        <min>0.1</min>
+                        <max>40</max>
+                        <resolution>0.01</resolution>
+                    </range>
+                    <noise>
+                        <type>gaussian</type>
+                        <mean>0.0</mean>
+                        <stddev>0.005</stddev>
+                    </noise>
+                </ray>
                 <plugin name="gazebo_ros_laser_controller" filename="liblivox_laser_simulation.so">
                     <ray>
@@ -336,42 +363,4 @@
             </sensor>
         </gazebo>
-        <!-- camera 单目相机插件 -->
-        <gazebo reference="front_camera">
-            <material>Gazebo/Grey</material>
-            <sensor type="camera" name="camera">
-                <update_rate>30.0</update_rate>
-                <camera name="head">
-                    <horizontal_fov>1.3962634</horizontal_fov>
-                    <image>
-                        <width>800</width>
-                        <height>800</height>
-                        <format>R8G8B8</format>
-                    </image>
-                    <clip>
-                        <near>0.02</near>
-                        <far>300</far>
-                    </clip>
-                    <noise>
-                        <type>gaussian</type>
-                        <mean>0.0</mean>
-                        <stddev>0.007</stddev>
-                    </noise>
-                </camera>
-                <plugin name="camera_controller" filename="libgazebo_ros_camera.so">
-                    <alwaysOn>true</alwaysOn>
-                    <updateRate>0.0</updateRate>
-                    <cameraName>camera</cameraName>
-                    <imageTopicName>image_raw</imageTopicName>
-                    <cameraInfoTopicName>camera_info</cameraInfoTopicName>
-                    <frameName>front_camera</frameName>
-                    <hackBaseline>0.07</hackBaseline>
-                    <distortionK1>0.0</distortionK1>
-                    <distortionK2>0.0</distortionK2>
-                    <distortionK3>0.0</distortionK3>
-                    <distortionT1>0.0</distortionT1>
-                    <distortionT2>0.0</distortionT2>
-                </plugin>
-            </sensor>
-        </gazebo>
         <!-- real_sense 深度相机(kinect)插件 -->
         <gazebo reference="real_sense">
@@ -400,5 +389,5 @@
                     <cameraInfoTopicName>rgb/camera_info</cameraInfoTopicName>
                     <depthImageCameraInfoTopicName>depth/camera_info</depthImageCameraInfoTopicName>
-                    <frameName>real_sense</frameName>
+                    <frameName>real_sense_optical_frame</frameName>
                     <baseline>0.1</baseline>
                     <distortion_k1>0.0</distortion_k1>

File: src/unitree_guide/unitree_ros/robots/a1_description/xacro/robot.xacro (robot description, xacro)
@@ -3,4 +3,5 @@
     <xacro:arg name="DEBUG" default="false"/>
     <xacro:arg name="ENABLE_SENSOR_DATA" default="true"/>
+    <xacro:arg name="ENABLE_FRONT_CAMERA" default="false"/>
     <xacro:arg name="ENABLE_GROUND_TRUTH" default="true"/>
     <xacro:arg name="ENABLE_FOOT_FORCE_VISUAL" default="false"/>
@@ -15,5 +16,5 @@
     <xacro:property name="rolloverProtection" value="false"/>
     <!-- Debug mode will hung up the robot, use "true" or "false" to switch it. -->
-    <xacro:if value="$(arg DEBUG)">
+    <xacro:if value="${'$(arg DEBUG)' == 'true'}">
         <link name="world"/>
         <joint name="base_static_joint" type="fixed">
@@ -193,4 +194,70 @@
             <axis xyz="0 0 1"/>
     </joint>
+    <link name="real_sense_optical_frame"/>
+    <joint name="real_sense_optical_joint" type="fixed">
+            <parent link="real_sense"/>
+            <child link="real_sense_optical_frame"/>
+            <!-- ROS optical frame: X right, Y down, Z forward. -->
+            <origin xyz="0 0 0" rpy="-1.57079632679 0 -1.57079632679"/>
+    </joint>
+    <xacro:if value="${'$(arg ENABLE_FRONT_CAMERA)' == 'true'}">
+        <!-- optional front monocular camera -->
+        <link name="front_camera">
+            <inertial>
+                <mass value="0.001"/>
+                <origin rpy="0 0 0" xyz="0 0 0"/>
+                <inertia ixx="0.0001" ixy="0" ixz="0" iyy="0.0001" iyz="0" izz="0.0001"/>
+            </inertial>
+            <visual>
+                <origin rpy="0 0 0" xyz="0 0 0"/>
+                <geometry>
+                    <box size="0.02 0.02 0.02"/>
+                </geometry>
+                <material name="black"/>
+            </visual>
+        </link>
+        <joint name="front_camera_joint" type="fixed">
+            <origin xyz="0.30 0 0.08" rpy="0 0 0"/>
+            <parent link="base"/>
+            <child link="front_camera"/>
+        </joint>
+        <gazebo reference="front_camera">
+            <material>Gazebo/Grey</material>
+            <sensor type="camera" name="camera">
+                <update_rate>30.0</update_rate>
+                <camera name="head">
+                    <horizontal_fov>1.3962634</horizontal_fov>
+                    <image>
+                        <width>800</width>
+                        <height>800</height>
+                        <format>R8G8B8</format>
+                    </image>
+                    <clip>
+                        <near>0.02</near>
+                        <far>300</far>
+                    </clip>
+                    <noise>
+                        <type>gaussian</type>
+                        <mean>0.0</mean>
+                        <stddev>0.007</stddev>
+                    </noise>
+                </camera>
+                <plugin name="camera_controller" filename="libgazebo_ros_camera.so">
+                    <alwaysOn>true</alwaysOn>
+                    <updateRate>0.0</updateRate>
+                    <cameraName>camera</cameraName>
+                    <imageTopicName>image_raw</imageTopicName>
+                    <cameraInfoTopicName>camera_info</cameraInfoTopicName>
+                    <frameName>front_camera</frameName>
+                    <hackBaseline>0.07</hackBaseline>
+                    <distortionK1>0.0</distortionK1>
+                    <distortionK2>0.0</distortionK2>
+                    <distortionK3>0.0</distortionK3>
+                    <distortionT1>0.0</distortionT1>
+                    <distortionT2>0.0</distortionT2>
+                </plugin>
+            </sensor>
+        </gazebo>
+    </xacro:if>
     <xacro:leg name="FR" mirror="-1" mirror_dae="False" front_hind="1" front_hind_dae="True">
         <origin rpy="0 0 0" xyz="${leg_offset_x} ${-leg_offset_y} 0"/>

Commit message: 解决实时率低

File: src/unitree_guide/unitree_ros/robots/a1_description/xacro/gazebo.xacro (robot description, xacro)
@@ -76,42 +76,44 @@
         <xacro:p3d_truth_plugin plugin_name="p3d_RR_foot_pos_vel" body_name="RR_foot" topic_name="ground_truth/RR_foot" frame_name="base"/>
     </xacro:if>
-    <!-- Foot contacts. -->
-    <gazebo reference="FR_calf">
-        <sensor name="FR_foot_contact" type="contact">
-        <update_rate>100</update_rate>
-        <plugin name="contactPlugin" filename="libunitreeFootContactPlugin.so"/>
-        <contact>
-            <collision>FR_calf_fixed_joint_lump__FR_foot_collision_1</collision>
-        </contact>
-        </sensor>
-    </gazebo>
-    <gazebo reference="FL_calf">
-        <sensor name="FL_foot_contact" type="contact">
-        <update_rate>100</update_rate>
-        <plugin name="contactPlugin" filename="libunitreeFootContactPlugin.so"/>
-        <contact>
-            <collision>FL_calf_fixed_joint_lump__FL_foot_collision_1</collision>
-        </contact>
-        </sensor>
-    </gazebo>
-    <gazebo reference="RR_calf">
-        <sensor name="RR_foot_contact" type="contact">
-        <update_rate>100</update_rate>
-        <plugin name="contactPlugin" filename="libunitreeFootContactPlugin.so"/>
-        <contact>
-            <collision>RR_calf_fixed_joint_lump__RR_foot_collision_1</collision>
-        </contact>
-        </sensor>
-    </gazebo>
-    <gazebo reference="RL_calf">
-        <sensor name="RL_foot_contact" type="contact">
-        <update_rate>100</update_rate>
-        <plugin name="contactPlugin" filename="libunitreeFootContactPlugin.so"/>
-        <contact>
-            <collision>RL_calf_fixed_joint_lump__RL_foot_collision_1</collision>
-        </contact>
-        </sensor>
-    </gazebo>
-    <xacro:if value="${'$(arg ENABLE_FOOT_FORCE_VISUAL)' == 'true'}">
+    <xacro:if value="${'$(arg ENABLE_FOOT_CONTACT_SENSOR)' == 'true'}">
+        <!-- Optional foot contact force topics. Disabling them keeps foot collisions unchanged. -->
+        <gazebo reference="FR_calf">
+            <sensor name="FR_foot_contact" type="contact">
+                <update_rate>100</update_rate>
+                <plugin name="contactPlugin" filename="libunitreeFootContactPlugin.so"/>
+                <contact>
+                    <collision>FR_calf_fixed_joint_lump__FR_foot_collision_1</collision>
+                </contact>
+            </sensor>
+        </gazebo>
+        <gazebo reference="FL_calf">
+            <sensor name="FL_foot_contact" type="contact">
+                <update_rate>100</update_rate>
+                <plugin name="contactPlugin" filename="libunitreeFootContactPlugin.so"/>
+                <contact>
+                    <collision>FL_calf_fixed_joint_lump__FL_foot_collision_1</collision>
+                </contact>
+            </sensor>
+        </gazebo>
+        <gazebo reference="RR_calf">
+            <sensor name="RR_foot_contact" type="contact">
+                <update_rate>100</update_rate>
+                <plugin name="contactPlugin" filename="libunitreeFootContactPlugin.so"/>
+                <contact>
+                    <collision>RR_calf_fixed_joint_lump__RR_foot_collision_1</collision>
+                </contact>
+            </sensor>
+        </gazebo>
+        <gazebo reference="RL_calf">
+            <sensor name="RL_foot_contact" type="contact">
+                <update_rate>100</update_rate>
+                <plugin name="contactPlugin" filename="libunitreeFootContactPlugin.so"/>
+                <contact>
+                    <collision>RL_calf_fixed_joint_lump__RL_foot_collision_1</collision>
+                </contact>
+            </sensor>
+        </gazebo>
+    </xacro:if>
+    <xacro:if value="${'$(arg ENABLE_FOOT_CONTACT_SENSOR)' == 'true' and '$(arg ENABLE_FOOT_FORCE_VISUAL)' == 'true'}">
         <!-- Visualization of foot contacts. Disabled by default for competition scenes. -->
         <gazebo reference="FR_foot">

File: src/unitree_guide/unitree_ros/robots/a1_description/xacro/robot.xacro (robot description, xacro)
@@ -5,4 +5,5 @@
     <xacro:arg name="ENABLE_FRONT_CAMERA" default="false"/>
     <xacro:arg name="ENABLE_GROUND_TRUTH" default="true"/>
+    <xacro:arg name="ENABLE_FOOT_CONTACT_SENSOR" default="false"/>
     <xacro:arg name="ENABLE_FOOT_FORCE_VISUAL" default="false"/>
     <xacro:include filename="$(find a1_description)/xacro/const.xacro"/>

Commit message: 可选传感器

File: src/unitree_guide/unitree_ros/robots/a1_description/xacro/gazebo.xacro (robot description, xacro)
@@ -274,7 +274,7 @@
         <kd  value="1.0"/>
     </gazebo>
-    <xacro:if value="${'$(arg ENABLE_SENSOR_DATA)' == 'true'}">
-        <!-- gazebo livox mid360 plugins -->
-        <xacro:property name="M_PI" value="3.14159"/>
+    <!-- gazebo livox mid360 plugins -->
+    <xacro:property name="M_PI" value="3.14159"/>
+    <xacro:if value="${'$(arg ENABLE_LIVOX)' == 'true'}">
         <gazebo reference="laser_livox">
             <sensor type="ray" name="laser_livox">
@@ -345,5 +345,7 @@
             </sensor>
         </gazebo>
-        <!-- gazebo livox imu-link plugins -->
+    </xacro:if>
+    <!-- gazebo livox imu-link plugins -->
+    <xacro:if value="${'$(arg ENABLE_LIVOX_IMU)' == 'true'}">
         <gazebo reference="livox_imu_link">
             <gravity>true</gravity>
@@ -365,5 +367,7 @@
             </sensor>
         </gazebo>
-        <!-- real_sense 深度相机(kinect)插件 -->
+    </xacro:if>
+    <!-- real_sense 深度相机(kinect)插件 -->
+    <xacro:if value="${'$(arg ENABLE_REALSENSE)' == 'true'}">
         <gazebo reference="real_sense">
             <sensor type="depth" name="real_sense">

File: src/unitree_guide/unitree_ros/robots/a1_description/xacro/robot.xacro (robot description, xacro)
@@ -3,4 +3,7 @@
     <xacro:arg name="DEBUG" default="false"/>
     <xacro:arg name="ENABLE_SENSOR_DATA" default="true"/>
+    <xacro:arg name="ENABLE_LIVOX" default="$(arg ENABLE_SENSOR_DATA)"/>
+    <xacro:arg name="ENABLE_LIVOX_IMU" default="$(arg ENABLE_LIVOX)"/>
+    <xacro:arg name="ENABLE_REALSENSE" default="$(arg ENABLE_SENSOR_DATA)"/>
     <xacro:arg name="ENABLE_FRONT_CAMERA" default="false"/>
     <xacro:arg name="ENABLE_GROUND_TRUTH" default="true"/>
