Commit message: 多层 demo 首次完整跑通：三层探索 + 三次换层 + 两次返程
mf61 = MISSION_COMPLETE。12 个房间全部探索，floor 0->1->2->0 三次换层，
二楼与三楼各一次上层返程，903.6 仿真秒。

修掉的八个阻塞项，每个都有实测证据：

1. 返程在点 C 多转 180 度导致坠楼（mf49）
   C 的 yaw 是走廊向外方向，直接当导航目标会让 MoveBase 在 C 转到背对 B，
   下一个 C->B 目标再转回来。bag: yaw 85.1->165.8->-161.9->129.6->71.3 度，
   DWA 在 wz -1.698 时已经 vx 0.409，横向偏离去程轨迹 0.32->0.77 m，
   真值 z 2.915->0.057。
   改：staging pose 保留 C 的 x/y、yaw 换成 atan2(B-C)；新增
   align_return_bearing_in_place() 在发目标前原地对正到零线速度。

2. 探索器与 mission 共用 /move_base 交接时无握手（mf51）
   ExploreFloor 返回瞬间发 goal 撞上 move_base 仍在 PREEMPTING，
   SimpleActionClient 状态机错乱，get_state() 返回 ACTIVE(1) 被当成终止状态。
   二楼报了一模一样的错却侥幸通过。
   改：settle_move_base_handover() 发 goal 前等 client 回到空闲。

3-6. 四处时间判据建立在没验算过的假设上
   - exploration wall_factor 5.0 假设 RTF 约 0.3，实测 0.165-0.272（mf53）
   - mission 五个墙钟兜底 factor 3.0-4.5，需 RTF > 0.22-0.33（mf54）
   - entry obstacle_hold_timeout 4 s 假设门是瞬时的，官方文档写明约 25 s，
     且 /set_door_state 只用 26 毫秒就返回（mf55）
   - action_timeout 纯墙钟 1800 s，是一层楼的探索总预算却按墙钟计（mf56）
   改：全部改为仿真预算 + 10 倍墙钟兜底（容忍 RTF 低到 0.10）；
   门等待改 30 仿真秒；新增 test_wall_clock_backstops.py 自动枚举所有配对、
   用实测最差 RTF 验算，并检查孤儿 *_sim。

7. 进轿厢的 A 平面后置条件是零容差（mf59）
   inset 0.40 < xy_goal_tolerance 0.45 且 latch_xy_goal_tolerance: true，
   所以 latch 后落点 = A + (-0.05 到 +0.40)，判据在最坏情况下不可满足。
   mf59 跑完全部三层探索后差 0.02 m 报废。
   改：upper_transfer_plane_tolerance 0.10，覆盖 -0.05 下界并留一倍余量，
   远小于本检查真正要防的 mf37（-0.361 m，机身仅 0.26 m 在开口内、横滚 96 度）。
   mf61 实测余量二楼 +0.034、三楼 +0.044。

8. 规划器暂不可用被当成房间已探完
   path_exists() 返回 None 时 break，落入完成分支并标记 proven；
   本该保护它的 if chosen is None 是死代码。
   改：置 planner_unavailable 后重试，预算耗尽留 unproven。

房间探索可观测性：
   room_transaction_frontiers 每一级都报 ROOM_FRONTIER_PIPELINE
   （map identity / 连通域 / ROI / keepout / raw / admissible）；
   选择循环报 ROOM_FRONTIER_SELECTION（score/visited/history/unreachable/
   planner_unavailable）；事务内发布房间候选 marker，绿线不再是进房前的快照。
   mf61 据此把「房间提前结束」分成两条独立路径各 7 次和 4 次。

demo 录像：接入 mission_video_recorder（第一人称 + 第三人称 + 未探索阴影），
   robot.xacro 加第三视角相机，绑 ENABLE_FRONT_CAMERA，默认关闭时展开 0 处。

返航：mission/final_return_to_start 默认 false。run() 尾部那段从电梯几何加
   2.3/3.5 m 硬编码重建起点的代码是占位实现，从未执行过，需等 backlog 第 2 节
   的 T_g 做出来。关闭时 exploration_time 不含返航段，不符合 PDF 定义，
   MISSION_COMPLETE 事件显式标注 return_to_start_performed=false。

已知未解决项见 ISSUE_LEDGER_问题台账.md（36 条，含被推翻的假设）。
危险源识别本轮未开启：跨层 world 坐标与 z 锚未解决前开了也拿不到分。

Co-Authored-By: Claude Opus 5 <noreply@anthropic.com>

File: src/unitree_guide/unitree_ros/robots/a1_description/xacro/robot.xacro (robot description, xacro)
@@ -263,4 +263,58 @@
             </sensor>
         </gazebo>
+        <!-- Optional over-shoulder camera for demo recording only. It is tied
+             to ENABLE_FRONT_CAMERA so auto.sh does not need another argument. -->
+        <link name="third_person_camera">
+            <inertial>
+                <mass value="0.001"/>
+                <origin rpy="0 0 0" xyz="0 0 0"/>
+                <inertia ixx="0.0001" ixy="0" ixz="0" iyy="0.0001" iyz="0" izz="0.0001"/>
+            </inertial>
+            <visual>
+                <origin rpy="0 0 0" xyz="0 0 0"/>
+                <geometry>
+                    <box size="0.02 0.02 0.02"/>
+                </geometry>
+                <material name="black"/>
+            </visual>
+        </link>
+        <joint name="third_person_camera_joint" type="fixed">
+            <origin xyz="-1.15 0 0.62" rpy="0 0.35 0"/>
+            <parent link="base"/>
+            <child link="third_person_camera"/>
+        </joint>
+        <gazebo reference="third_person_camera">
+            <material>Gazebo/Grey</material>
+            <sensor type="camera" name="third_person_camera">
+                <always_on>true</always_on>
+                <update_rate>12.0</update_rate>
+                <camera name="third_person">
+                    <horizontal_fov>1.15</horizontal_fov>
+                    <image>
+                        <width>640</width>
+                        <height>360</height>
+                        <format>R8G8B8</format>
+                    </image>
+                    <clip>
+                        <near>0.02</near>
+                        <far>60</far>
+                    </clip>
+                </camera>
+                <plugin name="third_person_camera_controller" filename="libgazebo_ros_camera.so">
+                    <alwaysOn>true</alwaysOn>
+                    <updateRate>0.0</updateRate>
+                    <cameraName>a1/third_person</cameraName>
+                    <imageTopicName>image_raw</imageTopicName>
+                    <cameraInfoTopicName>camera_info</cameraInfoTopicName>
+                    <frameName>third_person_camera</frameName>
+                    <hackBaseline>0.07</hackBaseline>
+                    <distortionK1>0.0</distortionK1>
+                    <distortionK2>0.0</distortionK2>
+                    <distortionK3>0.0</distortionK3>
+                    <distortionT1>0.0</distortionT1>
+                    <distortionT2>0.0</distortionT2>
+                </plugin>
+            </sensor>
+        </gazebo>
     </xacro:if>
     <xacro:leg name="FR" mirror="-1" mirror_dae="False" front_hind="1" front_hind_dae="True">
