Commit message: 初始化项目结构，附带结构说明MODULES.md

File: src/Mid360_imu_sim/urdf/livox_HAP.xacro (robot description, xacro)
@@ -15,5 +15,5 @@
     </inertial>
   </xacro:macro>
-  <xacro:macro name="Livox_Mid_gazebo_sensor" params="visualize:=True update_rate:=10 resolution:=0.002 noise_mean:=0.0 noise_stddev:=0.01 name:=livox">
+  <xacro:macro name="Livox_Mid_gazebo_sensor" params="visualize:=False update_rate:=10 resolution:=0.002 noise_mean:=0.0 noise_stddev:=0.01 name:=livox">
     <gazebo reference="${name}">
       <sensor type="ray" name="laser_${name}">
@@ -58,5 +58,5 @@
     </gazebo>
   </xacro:macro>
-  <xacro:macro name="Livox_Mid40" params="visualize:=True name:=livox">
+  <xacro:macro name="Livox_Mid40" params="visualize:=False name:=livox">
     <link name="${name}_base">
       <xacro:null_inertial/>

File: src/Mid360_imu_sim/urdf/livox_avia.xacro (robot description, xacro)
@@ -17,5 +17,5 @@
     </inertial>
   </xacro:macro>
-  <xacro:macro name="Livox_Mid_gazebo_sensor" params="visualize:=True update_rate:=10 resolution:=0.002 noise_mean:=0.0 noise_stddev:=0.01 name:=livox">
+  <xacro:macro name="Livox_Mid_gazebo_sensor" params="visualize:=False update_rate:=10 resolution:=0.002 noise_mean:=0.0 noise_stddev:=0.01 name:=livox">
     <gazebo reference="${name}">
       <sensor type="ray" name="laser_${name}">
@@ -60,5 +60,5 @@
     </gazebo>
   </xacro:macro>
-  <xacro:macro name="Livox_AVIA" params="visualize:=True name:=livox">
+  <xacro:macro name="Livox_AVIA" params="visualize:=False name:=livox">
     <link name="${name}_base">
       <xacro:null_inertial/>

File: src/Mid360_imu_sim/urdf/livox_horizon.xacro (robot description, xacro)
@@ -17,5 +17,5 @@
     </inertial>
   </xacro:macro>
-  <xacro:macro name="Livox_Mid_gazebo_sensor" params="visualize:=True update_rate:=10 resolution:=0.002 noise_mean:=0.0 noise_stddev:=0.01 name:=livox">
+  <xacro:macro name="Livox_Mid_gazebo_sensor" params="visualize:=False update_rate:=10 resolution:=0.002 noise_mean:=0.0 noise_stddev:=0.01 name:=livox">
     <gazebo reference="${name}">
       <sensor type="ray" name="laser_${name}">
@@ -60,5 +60,5 @@
     </gazebo>
   </xacro:macro>
-  <xacro:macro name="Livox_HORIZON" params="visualize:=True name:=livox">
+  <xacro:macro name="Livox_HORIZON" params="visualize:=False name:=livox">
     <link name="${name}_base">
       <xacro:null_inertial/>

File: src/Mid360_imu_sim/urdf/livox_mid360.xacro (robot description, xacro)
@@ -15,5 +15,5 @@
     </inertial>
   </xacro:macro>
-  <xacro:macro name="Livox_Mid_gazebo_sensor" params="visualize:=True update_rate:=10 resolution:=0.002 noise_mean:=0.0 noise_stddev:=0.01 name:=livox">
+  <xacro:macro name="Livox_Mid_gazebo_sensor" params="visualize:=False update_rate:=10 resolution:=0.002 noise_mean:=0.0 noise_stddev:=0.01 name:=livox">
     <gazebo reference="${name}">
       <sensor type="ray" name="laser_${name}">
@@ -58,5 +58,5 @@
     </gazebo>
   </xacro:macro>
-  <xacro:macro name="Livox_Mid40" params="visualize:=True name:=livox">
+  <xacro:macro name="Livox_Mid40" params="visualize:=False name:=livox">
     <link name="${name}_base">
       <xacro:null_inertial/>

File: src/Mid360_imu_sim/urdf/livox_mid40.xacro (robot description, xacro)
@@ -17,5 +17,5 @@
     </inertial>
   </xacro:macro>
-  <xacro:macro name="Livox_Mid_gazebo_sensor" params="visualize:=True update_rate:=10 resolution:=0.002 noise_mean:=0.0 noise_stddev:=0.01 name:=livox">
+  <xacro:macro name="Livox_Mid_gazebo_sensor" params="visualize:=False update_rate:=10 resolution:=0.002 noise_mean:=0.0 noise_stddev:=0.01 name:=livox">
     <gazebo reference="${name}">
       <sensor type="ray" name="laser_${name}">
@@ -60,5 +60,5 @@
     </gazebo>
   </xacro:macro>
-  <xacro:macro name="Livox_Mid40" params="visualize:=True name:=livox">
+  <xacro:macro name="Livox_Mid40" params="visualize:=False name:=livox">
     <link name="${name}_base">
       <xacro:null_inertial/>

File: src/Mid360_imu_sim/urdf/livox_mid70.xacro (robot description, xacro)
@@ -17,5 +17,5 @@
     </inertial>
   </xacro:macro>
-  <xacro:macro name="Livox_Mid_gazebo_sensor" params="visualize:=True update_rate:=10 resolution:=0.002 noise_mean:=0.0 noise_stddev:=0.01 name:=livox">
+  <xacro:macro name="Livox_Mid_gazebo_sensor" params="visualize:=False update_rate:=10 resolution:=0.002 noise_mean:=0.0 noise_stddev:=0.01 name:=livox">
     <gazebo reference="${name}">
       <sensor type="ray" name="laser_${name}">
@@ -60,5 +60,5 @@
     </gazebo>
   </xacro:macro>
-  <xacro:macro name="Livox_Mid70" params="visualize:=True name:=livox">
+  <xacro:macro name="Livox_Mid70" params="visualize:=False name:=livox">
     <link name="${name}_base">
       <xacro:null_inertial/>

File: src/Mid360_imu_sim/urdf/livox_tele.xacro (robot description, xacro)
@@ -17,5 +17,5 @@
     </inertial>
   </xacro:macro>
-  <xacro:macro name="Livox_Mid_gazebo_sensor" params="visualize:=True update_rate:=10 resolution:=0.002 noise_mean:=0.0 noise_stddev:=0.01 name:=livox">
+  <xacro:macro name="Livox_Mid_gazebo_sensor" params="visualize:=False update_rate:=10 resolution:=0.002 noise_mean:=0.0 noise_stddev:=0.01 name:=livox">
     <gazebo reference="${name}">
       <sensor type="ray" name="laser_${name}">
@@ -60,5 +60,5 @@
     </gazebo>
   </xacro:macro>
-  <xacro:macro name="Livox_TELE" params="visualize:=True name:=livox">
+  <xacro:macro name="Livox_TELE" params="visualize:=False name:=livox">
     <link name="${name}_base">
       <xacro:null_inertial/>

File: src/Mid360_imu_sim/urdf/mid360_IMU_platform.xacro (robot description, xacro)
@@ -74,5 +74,5 @@
                 <always_on>true</always_on>
                 <update_rate>200</update_rate>
-                <visualize>true</visualize>
+                <visualize>false</visualize>
                 <topic>/livox/imu</topic>
                 <plugin filename="libgazebo_ros_imu_sensor.so" name="imu_plugin">

File: src/unitree_guide/unitree_ros/robots/a1_description/xacro/gazebo.xacro (robot description, xacro)
@@ -281,5 +281,5 @@
                 <always_on>true</always_on>
                 <pose>0 0 0 0 0 0</pose>
-                <visualize>true</visualize>
+                <visualize>false</visualize>
                 <update_rate>10</update_rate>
                 <ray>
@@ -336,5 +336,5 @@
                         </noise>
                     </ray>
-                    <visualize>true</visualize>
+                    <visualize>false</visualize>
                     <samples>24000</samples>
                     <downsample>1</downsample>
